File: Projet/Alimentation.kicad_sch (KiCad schematic)
At the start: 13 parts

Commit message: board_schematic
Parts:
- removed J?: Screw_Terminal_01x02, symbol Connector:Screw_Terminal_01x02
- added J5001: alim batterie, Connector_JST:JST_XH_B2B-XH-A_1x02_P2.50mm_Vertical, symbol Connector_Generic:Conn_01x02
- added J?: pin verification, symbol Connector_Generic:Conn_01x01
- J5002: renamed from J?; value Conn_01x01 -> pin verification 5V
- J5003: renamed from J?; value Conn_01x01 -> pin verification 3.3V
- gave numbers to parts that had none: 10
Connections:
- net GND: now also J5001.2 (Pin_2), J?.1 (Pin_1)
- net V+_batterie: now also C5001.1, S5001.2, U5001.3 (VI); no longer S5001.3
- new net: J5001.1 (Pin_1), S5001.3
Other:
- note added: "mettre un label apres le switch resistance a dimensionner 100k"
- moved on the sheet: R5001, R5002, R5003, S5001

Commit message: pcb_begin
Parts:
- removed J5002: pin verification 5V, symbol Connector_Generic:Conn_01x01
- removed J5003: pin verification 3.3V, symbol Connector_Generic:Conn_01x01
- removed J?: pin verification, symbol Connector_Generic:Conn_01x01
- added J502: Conn_01x03_Female, Connector_PinHeader_2.54mm:PinHeader_1x03_P2.54mm_Vertical, symbol Connector:Conn_01x03_Female
- R501: renamed from R5003; value 100k -> 1k
- renumbered C5001 to C501, C5002 to C502, C5003 to C503, C5004 to C504, J5001 to J501, R5001 to R502, R5002 to R503, S5001 to S501, U5001 to U501, U5002 to U502
Connections:
- net +3.3V: now also J502.2 (Pin_2)
- net +5V: now also J502.1 (Pin_1)
- net GND: now also J502.3 (Pin_3)
Other:
- note added: "CHECK CONNECTOR"
- moved on the sheet: R502, R503

Commit message: placement
Changed lines of the file:
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@@
   (junction (at 128.27 87.63) (diameter 0) (color 0 0 0 0)
   )
+  (junction (at 163.83 101.346) (diameter 0) (color 0 0 0 0)
+  )
   (junction (at 163.83 99.06) (diameter 0) (color 0 0 0 0)
   )
@@
   (junction (at 101.6 87.63) (diameter 0) (color 0 0 0 0)
   )
-  (junction (at 163.83 101.854) (diameter 0) (color 0 0 0 0)
-  )
-  (junction (at 183.134 86.36) (diameter 0) (color 0 0 0 0)
+  (junction (at 184.912 86.36) (diameter 0) (color 0 0 0 0)
   )
   (junction (at 92.964 87.63) (diameter 0) (color 0 0 0 0)
@@
   (junction (at 180.34 86.36) (diameter 0) (color 0 0 0 0)
   )
+  (junction (at 94.742 67.31) (diameter 0) (color 0 0 0 0)
+  )
   (junction (at 149.86 86.36) (diameter 0) (color 0 0 0 0)
   )
@@
     (stroke (width 0) (type default) (color 0 0 0 0))
   )
-  (wire (pts (xy 181.356 79.502) (xy 181.356 81.28))
-    (stroke (width 0) (type default) (color 0 0 0 0))
-  )
   (wire (pts (xy 128.27 87.63) (xy 140.97 87.63))
     (stroke (width 0) (type default) (color 0 0 0 0))
@@
     (stroke (width 0) (type default) (color 0 0 0 0))
   )
+  (wire (pts (xy 202.692 101.346) (xy 163.83 101.346))
+    (stroke (width 0) (type default) (color 0 0 0 0))
+  )
   (polyline (pts (xy 191.77 110.49) (xy 135.89 110.49))
     (stroke (width 0) (type default) (color 0 0 0 0))
   )
+  (wire (pts (xy 218.186 57.404) (xy 184.912 57.404))
+    (stroke (width 0) (type default) (color 0 0 0 0))
+  )
   (wire (pts (xy 85.09 100.838) (xy 85.09 107.188))
     (stroke (width 0) (type default) (color 0 0 0 0))
@@
     (stroke (width 0) (type default) (color 0 0 0 0))
   )
+  (wire (pts (xy 94.742 54.864) (xy 94.742 67.31))
+    (stroke (width 0) (type default) (color 0 0 0 0))
+  )
   (wire (pts (xy 55.118 90.17) (xy 60.198 90.17))
     (stroke (width 0) (type default) (color 0 0 0 0))
@@
     (stroke (width 0) (type default) (color 0 0 0 0))
   )
+  (wire (pts (xy 218.186 54.864) (xy 94.742 54.864))
+    (stroke (width 0) (type default) (color 0 0 0 0))
+  )
   (polyline (pts (xy 60.198 78.74) (xy 60.198 92.71))
     (stroke (width 0) (type default) (color 0 0 0 0))
@@
     (stroke (width 0) (type default) (color 0 0 0 0))
   )
-  (wire (pts (xy 163.83 99.06) (xy 163.83 101.854))
+  (wire (pts (xy 163.83 99.06) (xy 163.83 101.346))
+    (stroke (width 0) (type default) (color 0 0 0 0))
+  )
+  (wire (pts (xy 202.692 59.944) (xy 202.692 101.346))
     (stroke (width 0) (type default) (color 0 0 0 0))
   )
@@
     (stroke (width 0) (type default) (color 0 0 0 0))
   )
-  (wire (pts (xy 163.83 101.854) (xy 163.83 102.87))
-    (stroke (width 0) (type default) (color 0 0 0 0))
-  )
   (wire (pts (xy 85.09 95.758) (xy 85.09 87.63))
     (stroke (width 0) (type default) (color 0 0 0 0))
@@
     (stroke (width 0) (type default) (color 0 0 0 0))
   )
-  (wire (pts (xy 68.58 67.31) (xy 128.27 67.31))
+  (wire (pts (xy 68.58 67.31) (xy 94.742 67.31))
     (stroke (width 0) (type default) (color 0 0 0 0))
   )
@@
     (stroke (width 0) (type default) (color 0 0 0 0))
   )
-  (wire (pts (xy 180.34 86.36) (xy 183.134 86.36))
-    (stroke (width 0) (type default) (color 0 0 0 0))
-  )
   (wire (pts (xy 55.118 96.52) (xy 55.118 97.79))
     (stroke (width 0) (type default) (color 0 0 0 0))
@@
     (stroke (width 0) (type default) (color 0 0 0 0))
   )
+  (wire (pts (xy 163.83 101.346) (xy 163.83 102.87))
+    (stroke (width 0) (type default) (color 0 0 0 0))
+  )
+  (wire (pts (xy 94.742 67.31) (xy 128.27 67.31))
+    (stroke (width 0) (type default) (color 0 0 0 0))
+  )
   (wire (pts (xy 153.67 86.36) (xy 149.86 86.36))
     (stroke (width 0) (type default) (color 0 0 0 0))
@@
     (stroke (width 0) (type default) (color 0 0 0 0))
   )
-  (wire (pts (xy 181.356 81.28) (xy 183.134 81.28))
-    (stroke (width 0) (type default) (color 0 0 0 0))
-  )
   (wire (pts (xy 33.02 83.82) (xy 33.02 87.122))
     (stroke (width 0) (type default) (color 0 0 0 0))
@@
     (stroke (width 0) (type default) (color 0 0 0 0))
   )
-  (wire (pts (xy 183.134 81.28) (xy 183.134 86.36))
+  (wire (pts (xy 184.912 57.404) (xy 184.912 86.36))
+    (stroke (width 0) (type default) (color 0 0 0 0))
+  )
+  (wire (pts (xy 184.912 86.36) (xy 194.31 86.36))
     (stroke (width 0) (type default) (color 0 0 0 0))
   )
@@
     (stroke (width 0) (type default) (color 0 0 0 0))
   )
-  (wire (pts (xy 163.068 101.854) (xy 163.83 101.854))
-    (stroke (width 0) (type default) (color 0 0 0 0))
-  )
-  (wire (pts (xy 183.134 86.36) (xy 194.31 86.36))
+  (wire (pts (xy 180.34 86.36) (xy 184.912 86.36))
     (stroke (width 0) (type default) (color 0 0 0 0))
   )
   (wire (pts (xy 101.6 87.63) (xy 101.6 88.9))
+    (stroke (width 0) (type default) (color 0 0 0 0))
+  )
+  (wire (pts (xy 218.186 59.944) (xy 202.692 59.944))
     (stroke (width 0) (type default) (color 0 0 0 0))
   )
@@
       (effects (font (size 1.27 1.27)) (justify right) hide)
     )
-  )
-  (global_label "alim5V" (shape input) (at 114.808 67.31 90) (fields_autoplaced)
-    (effects (font (size 1.27 1.27)) (justify left))
-    (property "Intersheet References" "${INTERSHEET_REFS}" (id 0) (at 114.7286 58.4864 90)
-      (effects (font (size 1.27 1.27)) (justify left) hide)
-    )
-  )
-  (global_label "GROUND" (shape input) (at 163.068 101.854 180) (fields_autoplaced)
-    (effects (font (size 1.27 1.27)) (justify right))
-    (property "Intersheet References" "${INTERSHEET_REFS}" (id 0) (at 152.8535 101.9334 0)
-      (effects (font (size 1.27 1.27)) (justify right) hide)
-    )
-  )
-  (global_label "GROUND" (shape input) (at 218.186 59.944 180) (fields_autoplaced)
-    (effects (font (size 1.27 1.27)) (justify right))
-    (property "Intersheet References" "${INTERSHEET_REFS}" (id 0) (at 207.9715 60.0234 0)
-      (effects (font (size 1.27 1.27)) (justify right) hide)
-    )
-  )
-  (global_label "alim3V" (shape input) (at 181.356 79.502 90) (fields_autoplaced)
-    (effects (font (size 1.27 1.27)) (justify left))
-    (property "Intersheet References" "${INTERSHEET_REFS}" (id 0) (at 181.2766 70.6784 90)
-      (effects (font (size 1.27 1.27)) (justify left) hide)
-    )
-  )
-  (global_label "alim3V" (shape input) (at 218.186 57.404 180) (fields_autoplaced)
-    (effects (font (size 1.27 1.27)) (justify right))
-    (property "Intersheet References" "${INTERSHEET_REFS}" (id 0) (at 209.3624 57.4834 0)
-      (effects (font (size 1.27 1.27)) (justify right) hide)
-    )
-  )
-  (global_label "alim5V" (shape input) (at 218.186 54.864 180) (fields_autoplaced)
-    (effects (font (size 1.27 1.27)) (justify right))
-    (property "Intersheet References" "${INTERSHEET_REFS}" (id 0) (at 209.3624 54.9434 0)
-      (effects (font (size 1.27 1.27)) (justify right) hide)
-    )

Commit message: Routing
Parts:
- C502: value 10uF -> 22uF
- R502: value 100k -> 200k
- R503: value 90k -> 100k
Other:
- note removed: "mettre un label apres le switch resistance a dimensionner 100k"
Changed lines of the file:
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@@
     (stroke (width 0) (type default) (color 0 0 0 0))
-  )
-  (text "mettre un label apres le switch\nresistance a dimensionner 100k\n"
-    (at 79.248 119.634 0)
-    (effects (font (size 1.27 1.27)) (justify left bottom))
   )
   (text "Regulateur 3.3 V" (at 157.48 72.39 0)
@@
       (effects (font (size 1.27 1.27)) (justify left))
     )
-    (property "Value" "10uF" (id 1) (at 130.81 92.7162 0)
+    (property "Value" "22uF" (id 1) (at 130.81 92.7162 0)
       (effects (font (size 1.27 1.27)) (justify left))
     )
@@
       (effects (font (size 1.27 1.27)) (justify right))
     )
-    (property "Value" "100k" (id 1) (at 87.63 99.5679 0)
+    (property "Value" "200k" (id 1) (at 87.63 99.5679 0)
       (effects (font (size 1.27 1.27)) (justify right))
     )
@@
       (effects (font (size 1.27 1.27)) (justify right))
     )
-    (property "Value" "90k" (id 1) (at 87.63 110.9979 0)
-      (effects (font (size 1.27 1.27)) (justify right))
-    )
+    (property "Value" "100k" (id 1) (at 87.63 110.9979 0)
+      (effects (font (size 1.27 1.27)) (justify right))
+    )

Commit message: PCB_Modif2
Parts:
- removed U501: AZ1117-5.0, Package_TO_SOT_SMD:SOT-223-3_TabPin2, symbol Regulator_Linear:AZ1117-5.0
- removed U502: MIC5317-3.3, Package_TO_SOT_SMD:SOT-23-5, symbol Regulator_Linear:MCP1802x-xx02xOT
- added IC?: AZ1117CH2-5.0TRG1, AZ1117CH2:SOT230P700X180-4N, symbol AZ1117CH2-5.0TRG1:AZ1117CH2-5.0TRG1
- added PS?: MIC5317-3.3YM5-TR, MIC5317:SOT95P280X145-5N, symbol MIC5317-3.3YM5-TR:MIC5317-3.3YM5-TR
Connections:
- net +3.3V: now also PS?.5 (VOUT)
- net +5V: now also IC?.3 (OUTPUT), PS?.1 (VIN), PS?.3 (EN)
- net GND: now also IC?.2 (ADJ/GND_1), IC?.4 (ADJ/GND_2), PS?.2 (GND)
- net V+_batterie: now also IC?.1 (INPUT)
Other:
- moved on the sheet: C503, C504

Commit message: Routage_fini
Parts:
- removed S501: Alimentation, SWITCH_PRO:SW_100SP1T1B4M2QE, symbol SWITCH_PRO:100SP1T1B4M2QE
- added S501: 100SP1T1B4M2QE, SW_100SP1T1B4M2QE, symbol 100SP1T1B4M2QE:100SP1T1B4M2QE
- gave numbers to parts that had none: 2
Connections:
- net V+_batterie: now also S501.2
- net at R501.2: now also S501.1
- net at J501.1 (Pin_1): now also S501.3
Changed lines of the file:
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@@
     (stroke (width 0) (type default) (color 0 0 0 0))
   )
-  (wire (pts (xy 49.53 85.09) (xy 60.198 85.09))
+  (wire (pts (xy 49.53 85.09) (xy 60.452 85.09))
     (stroke (width 0) (type default) (color 0 0 0 0))
   )
@@
     (stroke (width 0) (type default) (color 0 0 0 0))
   )
-  (wire (pts (xy 55.118 90.17) (xy 60.198 90.17))
+  (wire (pts (xy 55.118 90.17) (xy 60.452 90.17))
     (stroke (width 0) (type default) (color 0 0 0 0))
   )
@@
     (stroke (width 0) (type default) (color 0 0 0 0))
   )
-  (wire (pts (xy 75.438 87.63) (xy 85.09 87.63))
+  (wire (pts (xy 75.692 87.63) (xy 85.09 87.63))
     (stroke (width 0) (type default) (color 0 0 0 0))
   )
@@
   (symbol (lib_id "power:+5V") (at 147.574 74.93 0) (unit 1)
     (in_bom yes) (on_board yes) (fields_autoplaced)
-    (property "Reference" "#PWR?" (id 0) (at 147.574 78.74 0)
+    (property "Reference" "#PWR0115" (id 0) (at 147.574 78.74 0)
       (effects (font (size 1.27 1.27)) hide)
     )
@@
     (pin "1")
   )
-  (symbol (lib_id "SWITCH_PRO:100SP1T1B4M2QE") (at 67.818 87.63 180) (unit 1)
-    (in_bom yes) (on_board yes)
-    (property "Reference" "S501" (id 0) (at 67.818 80.01 0))
-    (property "Value" "Alimentation" (id 1) (at 67.818 82.55 0))
-    (property "Footprint" "SWITCH_PRO:SW_100SP1T1B4M2QE" (id 2) (at 67.818 87.63 0)
-      (effects (font (size 1.27 1.27)) (justify left bottom) hide)
-    )
-    (property "Datasheet" "" (id 3) (at 67.818 87.63 0)
-      (effects (font (size 1.27 1.27)) (justify left bottom) hide)
-    )
-    (property "MAXIMUM_PACKAGE_HEIGHT" "29.68 mm" (id 4) (at 67.818 87.63 0)
-      (effects (font (size 1.27 1.27)) (justify left bottom) hide)
-    )
-    (property "STANDARD" "Manufacturer Recommendations" (id 5) (at 67.818 87.63 0)
-      (effects (font (size 1.27 1.27)) (justify left bottom) hide)
-    )
-    (property "MANUFACTURER" "E-Switch" (id 6) (at 67.818 87.63 0)
-      (effects (font (size 1.27 1.27)) (justify left bottom) hide)
-    )
-    (property "PARTREV" "E" (id 7) (at 67.818 87.63 0)
-      (effects (font (size 1.27 1.27)) (justify left bottom) hide)
-    )
-    (pin "1")
-    (pin "2")
-    (pin "3")
-  )
   (symbol (lib_id "power:+3.3V") (at 214.63 86.106 0) (unit 1)
     (in_bom yes) (on_board yes) (fields_autoplaced)
@@
   (symbol (lib_id "AZ1117CH2-5.0TRG1:AZ1117CH2-5.0TRG1") (at 107.188 76.962 90) (unit 1)
     (in_bom yes) (on_board yes) (fields_autoplaced)
-    (property "Reference" "IC?" (id 0) (at 115.57 55.3719 90)
+    (property "Reference" "IC501" (id 0) (at 115.57 55.3719 90)
       (effects (font (size 1.27 1.27)) (justify right))
     )
@@
     (pin "1")
   )
+  (symbol (lib_id "100SP1T1B4M2QE:100SP1T1B4M2QE") (at 68.072 87.63 180) (unit 1)
+    (in_bom yes) (on_board yes) (fields_autoplaced)
+    (property "Reference" "S501" (id 0) (at 68.072 80.01 0))
+    (property "Value" "100SP1T1B4M2QE" (id 1) (at 68.072 82.55 0))
+    (property "Footprint" "SW_100SP1T1B4M2QE" (id 2) (at 68.072 87.63 0)
+      (effects (font (size 1.27 1.27)) (justify left bottom) hide)
+    )
+    (property "Datasheet" "" (id 3) (at 68.072 87.63 0)
+      (effects (font (size 1.27 1.27)) (justify left bottom) hide)
+    )
+    (property "MAXIMUM_PACKAGE_HEIGHT" "29.68 mm" (id 4) (at 68.072 87.63 0)
+      (effects (font (size 1.27 1.27)) (justify left bottom) hide)
+    )
+    (property "STANDARD" "Manufacturer Recommendations" (id 5) (at 68.072 87.63 0)
+      (effects (font (size 1.27 1.27)) (justify left bottom) hide)
+    )
+    (property "MANUFACTURER" "E-Switch" (id 6) (at 68.072 87.63 0)
+      (effects (font (size 1.27 1.27)) (justify left bottom) hide)
+    )
+    (property "PARTREV" "E" (id 7) (at 68.072 87.63 0)
+      (effects (font (size 1.27 1.27)) (justify left bottom) hide)
+    )
+    (pin "1")
+    (pin "2")
+    (pin "3")
+  )
   (symbol (lib_id "Device:C_Small") (at 101.6 91.44 0) (unit 1)
     (in_bom yes) (on_board yes) (fields_autoplaced)
@@
   (symbol (lib_id "power:GND") (at 138.176 42.672 0) (unit 1)
     (in_bom yes) (on_board yes) (fields_autoplaced)
-    (property "Reference" "#PWR?" (id 0) (at 138.176 49.022 0)
+    (property "Reference" "#PWR0114" (id 0) (at 138.176 49.022 0)
       (effects (font (size 1.27 1.27)) hide)
     )
@@
   (symbol (lib_id "MIC5317-3.3YM5-TR:MIC5317-3.3YM5-TR") (at 167.64 80.772 0) (unit 1)
     (in_bom yes) (on_board yes) (fields_autoplaced)
-    (property "Reference" "PS?" (id 0) (at 181.61 72.898 0))
+    (property "Reference" "PS501" (id 0) (at 181.61 72.898 0))
     (property "Value" "MIC5317-3.3YM5-TR" (id 1) (at 181.61 75.438 0))
     (property "Footprint" "MIC5317:SOT95P280X145-5N" (id 2) (at 191.77 78.232 0)
@@
   (symbol (lib_id "power:GND") (at 216.408 59.944 0) (unit 1)
     (in_bom yes) (on_board yes) (fields_autoplaced)
-    (property "Reference" "#PWR?" (id 0) (at 216.408 66.294 0)
+    (property "Reference" "#PWR0117" (id 0) (at 216.408 66.294 0)
       (effects (font (size 1.27 1.27)) hide)
     )
@@
   (symbol (lib_id "power:+5V") (at 165.862 85.852 90) (unit 1)
     (in_bom yes) (on_board yes)
-    (property "Reference" "#PWR?" (id 0) (at 169.672 85.852 0)
-      (effects (font (size 1.27 1.27)) hide)
-    )
+    (property "Reference" "#PWR0116" (id 0) (at 169.672 85.852 0)
+      (effects (font (size 1.27 1.27)) hide)
+    )
