File: Projet/Projet.kicad_pcb (KiCad board)
At the start: 4 copper layers, 137.1 x 57 mm, 76 parts, among them IC501 AZ1117CH2-5.0TRG1, J201 Conn_02x07_Odd_Even, J301 Moteur 2, J302 Moteur 1, J303 Conn_01x03, J401 optiqueGauche, J402 couleursGauche, J403 couleursDroit, J404 optiqueDroit, J405 tofDroit, J406 tofGauche, J501 alim batterie, J502 Conn_01x03_Female, U201 STM32G070RBT6, U301 ZXBM5210-S, U302 ZXBM5210-S, Y201 16 MHz

Commit message: Routage_Final
Connections:
- J402 pad 4: unconnected-(J402-Pad4) -> /STM32F070RB/CLR_LED
- J402 pad 5: unconnected-(J402-Pad5) -> GND
- U201 pad 58: unconnected-(U201-Pad58) -> /STM32F070RB/CLR_LED
Routing:
- net /STM32F070RB/CLR_LED: track 0.00 -> 23.7 mm, vias 0 -> 2
- net +5V: track 99.6 -> 104.4 mm, vias 7 -> 8

Commit message: PCB_FINAL
Parts:
- removed A601: Adafruit_Feather_HUZZAH32_ESP32, Module:Adafruit_Feather
- removed C205: 100nF, Capacitor_SMD:C_0603_1608Metric_Pad1.08x0.95mm_HandSolder
- removed JP301, JP302: SolderJumper_2_Open, Jumper:SolderJumper-2_P1.3mm_Open_TrianglePad1.0x1.5mm
- added G1: LOGO, Logo_ensea:ENSEA_LOGO, F.Cu at (123.2, 127.8)
- added J601: Conn_01x04_Female, Connector_JST:JST_XH_B4B-XH-A_1x04_P2.50mm_Vertical, F.Cu at (200.8, 133.2)
- moved R301 28.1 mm to (154.8, 131.7), turned to 180 degrees
- moved C304 26.1 mm to (172.7, 138.1), turned to 0 degrees
- moved C306 21.1 mm to (169.8, 140.7), turned to -90 degrees
- moved JP304 21.1 mm to (167.4, 140.7), turned to -90 degrees
- moved C202 16.5 mm to (143.8, 123.0)
- moved R203 15.8 mm to (147.0, 125.7)
- moved Y201 15.7 mm to (146.9, 123.0)
- moved C502 11.6 mm to (107.3, 117.6), turned to 180 degrees
- moved C203 10.5 mm to (147.1, 120.0), turned to 180 degrees
- moved C301 9.88 mm to (107.0, 126.0)
- moved C501 8.91 mm to (107.4, 112.1), turned to 90 degrees
- moved JP305 8.01 mm to (138.1, 141.4), turned to -90 degrees
- moved C307 6.98 mm to (135.2, 128.8), turned to 90 degrees
- moved C201 5.72 mm to (190.6, 109.3), turned to -90 degrees
- moved R501 5.48 mm to (104.6, 129.9)
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Connections:
- net Net-(C203-Pad1) renamed /STM32F070RB/OSC_IN
- net Net-(R203-Pad1) renamed /STM32F070RB/OSC_OUT
- C303 pad 1: /Driver_Motor_SERVO/5V_DRV_2 -> +5V
- C304 pad 1: /Driver_Motor_SERVO/5V_DRV_1 -> +5V
- U201 pad 1: unconnected-(U201-Pad1) -> /STM32F070RB/OPTQ1
- U201 pad 14: /STM32F070RB/OPTQ1 -> unconnected-(U201-Pad14)
- U201 pad 21: /Communication/ESP_EN -> unconnected-(U201-Pad21)
- U301 pad 3: /Driver_Motor_SERVO/5V_DRV_2 -> +5V
- U301 pad 6: unconnected-(U301-Pad6) -> +5V
- U302 pad 3: /Driver_Motor_SERVO/5V_DRV_1 -> +5V
Routing:
- net /Communication/ESP_EN: track 86.0 -> 0.00 mm, vias 2 -> 0
- net /Driver_Motor_SERVO/5V_DRV_1: track 39.9 -> 0.00 mm, vias 2 -> 0
- net GND: track 11.2 -> 33.9 mm, vias 6 -> 12
- net /Driver_Motor_SERVO/VM_DRIVER_1_JP: track 28.2 -> 6.77 mm, vias 2 -> 0
- net /STM32F070RB/NRST_sw: track 71.4 -> 52.5 mm
- net +5V: track 104.4 -> 122.1 mm, vias 8 -> 7
- net /STM32F070RB/OSC_IN: track 21.7 -> 5.77 mm
- net /STM32F070RB/OSC_OUT: track 23.0 -> 7.69 mm, vias 2 -> 0
- net /Driver_Motor_SERVO/5V_DRV_2: track 13.7 -> 0.00 mm
- net V+_batterie: track 63.8 -> 54.9 mm
- net /STM32F070RB/OPTQ1: track 61.9 -> 53.5 mm, vias 2 -> 0
- net /Communication/ESP_TX_JP: track 56.8 -> 49.1 mm
- net /Driver_Motor_SERVO/SERV_DATA: track 54.5 -> 47.3 mm, vias 2 -> 3
- net /Driver_Motor_SERVO/M2+_JP: track 12.7 -> 5.83 mm
- net /Driver_Motor_SERVO/M2-_JP: track 32.9 -> 26.3 mm
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Other:
- board size 137.1 x 57 mm -> 113.1 x 57 mm
- board text added: "5V"
- board text added: "ESP"
