File: Projet/_autosave-Driver_Motor.kicad_sch (KiCad schematic)
At the start: 22 parts, among them J301 Moteur 2, J302 Moteur 1, J303 Conn_01x03, U301 ZXBM5210-S, U302 ZXBM5210-S

Commit message: PCB_FINAL
Changed lines of the file:
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@@
     (stroke (width 0) (type default) (color 0 0 0 0))
   )
-  (wire (pts (xy 67.056 39.116) (xy 64.77 39.116))
+  (wire (pts (xy 67.818 39.116) (xy 64.77 39.116))
     (stroke (width 0) (type default) (color 0 0 0 0))
   )
@@
     (pin "2")
   )
-  (symbol (lib_id "power:GND") (at 67.056 39.116 0) (unit 1)
-    (in_bom yes) (on_board yes) (fields_autoplaced)
-    (property "Reference" "#PWR0311" (id 0) (at 67.056 45.466 0)
-      (effects (font (size 1.27 1.27)) hide)
-    )
-    (property "Value" "GND" (id 1) (at 67.056 44.45 0))
-    (property "Footprint" "" (id 2) (at 67.056 39.116 0)
-      (effects (font (size 1.27 1.27)) hide)
-    )
-    (property "Datasheet" "" (id 3) (at 67.056 39.116 0)
-      (effects (font (size 1.27 1.27)) hide)
-    )
+  (symbol (lib_id "power:GND") (at 67.818 39.116 0) (unit 1)
+    (in_bom yes) (on_board yes) (fields_autoplaced)
+    (property "Reference" "#PWR0311" (id 0) (at 67.818 45.466 0)
+      (effects (font (size 1.27 1.27)) hide)
+    )
+    (property "Value" "GND" (id 1) (at 67.818 44.45 0))
+    (property "Footprint" "" (id 2) (at 67.818 39.116 0)
+      (effects (font (size 1.27 1.27)) hide)
+    )
+    (property "Datasheet" "" (id 3) (at 67.818 39.116 0)
+      (effects (font (size 1.27 1.27)) hide)
+    )
