File: Projet/bloc_capteur.kicad_sch (KiCad schematic)
At the start: 8 parts

Commit message: board_schematic
Parts:
- gave numbers to parts that had none: 8
Changed lines of the file:
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@@
   (symbol (lib_id "Connector:Conn_01x03_Female") (at 59.69 166.37 0) (unit 1)
     (in_bom yes) (on_board yes) (fields_autoplaced)
-    (property "Reference" "J?" (id 0) (at 60.96 165.0999 0)
+    (property "Reference" "J4001" (id 0) (at 60.96 165.0999 0)
       (effects (font (size 1.27 1.27)) (justify left))
     )
@@
   (symbol (lib_id "power:+3.3V") (at 57.15 57.15 90) (unit 1)
     (in_bom yes) (on_board yes)
-    (property "Reference" "#PWR?" (id 0) (at 60.96 57.15 0)
+    (property "Reference" "#PWR0128" (id 0) (at 60.96 57.15 0)
       (effects (font (size 1.27 1.27)) hide)
     )
@@
   (symbol (lib_id "Connector:Conn_01x03_Female") (at 106.68 167.64 0) (mirror y) (unit 1)
     (in_bom yes) (on_board yes) (fields_autoplaced)
-    (property "Reference" "J?" (id 0) (at 105.41 166.3699 0)
+    (property "Reference" "J4004" (id 0) (at 105.41 166.3699 0)
       (effects (font (size 1.27 1.27)) (justify left))
     )
@@
   (symbol (lib_id "Connector:Conn_01x07_Female") (at 212.09 63.5 0) (unit 1)
     (in_bom yes) (on_board yes) (fields_autoplaced)
-    (property "Reference" "J?" (id 0) (at 213.36 62.2299 0)
+    (property "Reference" "J4005" (id 0) (at 213.36 62.2299 0)
       (effects (font (size 1.27 1.27)) (justify left))
     )
@@
   (symbol (lib_id "Device:C_Small") (at 41.91 163.83 0) (unit 1)
     (in_bom yes) (on_board yes) (fields_autoplaced)
-    (property "Reference" "C?" (id 0) (at 44.45 162.5662 0)
+    (property "Reference" "C4001" (id 0) (at 44.45 162.5662 0)
       (effects (font (size 1.27 1.27)) (justify left))
     )
@@
   (symbol (lib_id "Connector:Conn_01x05_Female") (at 62.23 62.23 0) (unit 1)
     (in_bom yes) (on_board yes)
-    (property "Reference" "J?" (id 0) (at 63.5 60.9599 0)
+    (property "Reference" "J4002" (id 0) (at 63.5 60.9599 0)
       (effects (font (size 1.27 1.27)) (justify left))
     )
@@
   (symbol (lib_id "power:+3.3V") (at 133.35 167.64 270) (mirror x) (unit 1)
     (in_bom yes) (on_board yes) (fields_autoplaced)
-    (property "Reference" "#PWR?" (id 0) (at 129.54 167.64 0)
+    (property "Reference" "#PWR0129" (id 0) (at 129.54 167.64 0)
       (effects (font (size 1.27 1.27)) hide)
     )
@@
   (symbol (lib_id "power:GND") (at 242.57 60.96 90) (mirror x) (unit 1)
     (in_bom yes) (on_board yes) (fields_autoplaced)
-    (property "Reference" "#PWR?" (id 0) (at 248.92 60.96 0)
+    (property "Reference" "#PWR0132" (id 0) (at 248.92 60.96 0)
       (effects (font (size 1.27 1.27)) hide)
     )
@@
   (symbol (lib_id "power:GND") (at 207.01 60.96 270) (unit 1)
     (in_bom yes) (on_board yes) (fields_autoplaced)
-    (property "Reference" "#PWR?" (id 0) (at 200.66 60.96 0)
+    (property "Reference" "#PWR0130" (id 0) (at 200.66 60.96 0)
       (effects (font (size 1.27 1.27)) hide)
     )
@@
   (symbol (lib_id "Connector:Conn_01x05_Female") (at 78.74 62.23 180) (unit 1)
     (in_bom yes) (on_board yes)
-    (property "Reference" "J?" (id 0) (at 77.47 63.5001 0)
+    (property "Reference" "J4003" (id 0) (at 77.47 63.5001 0)
       (effects (font (size 1.27 1.27)) (justify left))
     )
@@
   (symbol (lib_id "power:GND") (at 57.15 59.69 270) (unit 1)
     (in_bom yes) (on_board yes) (fields_autoplaced)
-    (property "Reference" "#PWR?" (id 0) (at 50.8 59.69 0)
+    (property "Reference" "#PWR0127" (id 0) (at 50.8 59.69 0)
       (effects (font (size 1.27 1.27)) hide)
     )
@@
   (symbol (lib_id "power:GND") (at 133.35 162.56 90) (mirror x) (unit 1)
     (in_bom yes) (on_board yes) (fields_autoplaced)
-    (property "Reference" "#PWR?" (id 0) (at 139.7 162.56 0)
+    (property "Reference" "#PWR0126" (id 0) (at 139.7 162.56 0)
       (effects (font (size 1.27 1.27)) hide)
     )
@@
   (symbol (lib_id "Device:C_Small") (at 120.65 165.1 0) (unit 1)
     (in_bom yes) (on_board yes) (fields_autoplaced)
-    (property "Reference" "C?" (id 0) (at 123.19 163.8362 0)
+    (property "Reference" "C4002" (id 0) (at 123.19 163.8362 0)
       (effects (font (size 1.27 1.27)) (justify left))
     )
@@
   (symbol (lib_id "power:+3.3V") (at 207.01 58.42 90) (unit 1)
     (in_bom yes) (on_board yes) (fields_autoplaced)
-    (property "Reference" "#PWR?" (id 0) (at 210.82 58.42 0)
+    (property "Reference" "#PWR0131" (id 0) (at 210.82 58.42 0)
       (effects (font (size 1.27 1.27)) hide)
     )
@@
   (symbol (lib_id "power:+3.3V") (at 242.57 58.42 270) (mirror x) (unit 1)
     (in_bom yes) (on_board yes) (fields_autoplaced)
-    (property "Reference" "#PWR?" (id 0) (at 238.76 58.42 0)
+    (property "Reference" "#PWR0133" (id 0) (at 238.76 58.42 0)
       (effects (font (size 1.27 1.27)) hide)
     )
@@
   (symbol (lib_id "power:+3.3V") (at 35.56 166.37 90) (unit 1)
     (in_bom yes) (on_board yes) (fields_autoplaced)
-    (property "Reference" "#PWR?" (id 0) (at 39.37 166.37 0)
+    (property "Reference" "#PWR0124" (id 0) (at 39.37 166.37 0)
       (effects (font (size 1.27 1.27)) hide)
     )
@@
   (symbol (lib_id "Connector:Conn_01x07_Female") (at 237.49 63.5 0) (mirror y) (unit 1)
     (in_bom yes) (on_board yes)
-    (property "Reference" "J?" (id 0) (at 231.14 62.23 0))
+    (property "Reference" "J4006" (id 0) (at 231.14 62.23 0))
     (property "Value" "tofDroit" (id 1) (at 231.14 64.77 0))
     (property "Footprint" "Connector_JST:JST_XH_B7B-XH-A_1x07_P2.50mm_Vertical" (id 2) (at 237.49 63.5 0)
@@
   (symbol (lib_id "power:GND") (at 35.56 161.29 270) (unit 1)
     (in_bom yes) (on_board yes) (fields_autoplaced)
-    (property "Reference" "#PWR?" (id 0) (at 29.21 161.29 0)
-      (effects (font (size 1.27 1.27)) hide)
-    )
+    (property "Reference" "#PWR0125" (id 0) (at 29.21 161.29 0)
+      (effects (font (size 1.27 1.27)) hide)
+    )

Commit message: pcb_begin
Parts:
- J402: renamed from J4002; value couleursGauche -> couleursDroit
- renumbered C4001 to C401, C4002 to C402, J4001 to J401, J4003 to J403, J4004 to J404, J4005 to J405, J4006 to J406
Changed lines of the file:
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@@
   (symbol (lib_id "Connector:Conn_01x03_Female") (at 59.69 166.37 0) (unit 1)
     (in_bom yes) (on_board yes) (fields_autoplaced)
-    (property "Reference" "J4001" (id 0) (at 60.96 165.0999 0)
+    (property "Reference" "J401" (id 0) (at 60.96 165.0999 0)
       (effects (font (size 1.27 1.27)) (justify left))
     )
@@
   (symbol (lib_id "power:+3.3V") (at 57.15 57.15 90) (unit 1)
     (in_bom yes) (on_board yes)
-    (property "Reference" "#PWR0128" (id 0) (at 60.96 57.15 0)
+    (property "Reference" "#PWR0403" (id 0) (at 60.96 57.15 0)
       (effects (font (size 1.27 1.27)) hide)
     )
@@
   (symbol (lib_id "Connector:Conn_01x03_Female") (at 106.68 167.64 0) (mirror y) (unit 1)
     (in_bom yes) (on_board yes) (fields_autoplaced)
-    (property "Reference" "J4004" (id 0) (at 105.41 166.3699 0)
+    (property "Reference" "J404" (id 0) (at 105.41 166.3699 0)
       (effects (font (size 1.27 1.27)) (justify left))
     )
@@
   (symbol (lib_id "Connector:Conn_01x07_Female") (at 212.09 63.5 0) (unit 1)
     (in_bom yes) (on_board yes) (fields_autoplaced)
-    (property "Reference" "J4005" (id 0) (at 213.36 62.2299 0)
+    (property "Reference" "J405" (id 0) (at 213.36 62.2299 0)
       (effects (font (size 1.27 1.27)) (justify left))
     )
@@
   (symbol (lib_id "Device:C_Small") (at 41.91 163.83 0) (unit 1)
     (in_bom yes) (on_board yes) (fields_autoplaced)
-    (property "Reference" "C4001" (id 0) (at 44.45 162.5662 0)
+    (property "Reference" "C401" (id 0) (at 44.45 162.5662 0)
       (effects (font (size 1.27 1.27)) (justify left))
     )
@@
   (symbol (lib_id "Connector:Conn_01x05_Female") (at 62.23 62.23 0) (unit 1)
     (in_bom yes) (on_board yes)
-    (property "Reference" "J4002" (id 0) (at 63.5 60.9599 0)
-      (effects (font (size 1.27 1.27)) (justify left))
-    )
-    (property "Value" "couleursGauche" (id 1) (at 53.34 53.34 0)
+    (property "Reference" "J402" (id 0) (at 63.5 60.9599 0)
+      (effects (font (size 1.27 1.27)) (justify left))
+    )
+    (property "Value" "couleursDroit" (id 1) (at 53.34 53.34 0)
       (effects (font (size 1.27 1.27)) (justify left))
     )
@@
   (symbol (lib_id "power:+3.3V") (at 133.35 167.64 270) (mirror x) (unit 1)
     (in_bom yes) (on_board yes) (fields_autoplaced)
-    (property "Reference" "#PWR0129" (id 0) (at 129.54 167.64 0)
+    (property "Reference" "#PWR0406" (id 0) (at 129.54 167.64 0)
       (effects (font (size 1.27 1.27)) hide)
     )
@@
   (symbol (lib_id "power:GND") (at 242.57 60.96 90) (mirror x) (unit 1)
     (in_bom yes) (on_board yes) (fields_autoplaced)
-    (property "Reference" "#PWR0132" (id 0) (at 248.92 60.96 0)
+    (property "Reference" "#PWR0410" (id 0) (at 248.92 60.96 0)
       (effects (font (size 1.27 1.27)) hide)
     )
@@
   (symbol (lib_id "power:GND") (at 207.01 60.96 270) (unit 1)
     (in_bom yes) (on_board yes) (fields_autoplaced)
-    (property "Reference" "#PWR0130" (id 0) (at 200.66 60.96 0)
+    (property "Reference" "#PWR0408" (id 0) (at 200.66 60.96 0)
       (effects (font (size 1.27 1.27)) hide)
     )
@@
   (symbol (lib_id "Connector:Conn_01x05_Female") (at 78.74 62.23 180) (unit 1)
     (in_bom yes) (on_board yes)
-    (property "Reference" "J4003" (id 0) (at 77.47 63.5001 0)
+    (property "Reference" "J403" (id 0) (at 77.47 63.5001 0)
       (effects (font (size 1.27 1.27)) (justify left))
     )
@@
   (symbol (lib_id "power:GND") (at 57.15 59.69 270) (unit 1)
     (in_bom yes) (on_board yes) (fields_autoplaced)
-    (property "Reference" "#PWR0127" (id 0) (at 50.8 59.69 0)
+    (property "Reference" "#PWR0404" (id 0) (at 50.8 59.69 0)
       (effects (font (size 1.27 1.27)) hide)
     )
@@
   (symbol (lib_id "power:GND") (at 133.35 162.56 90) (mirror x) (unit 1)
     (in_bom yes) (on_board yes) (fields_autoplaced)
-    (property "Reference" "#PWR0126" (id 0) (at 139.7 162.56 0)
+    (property "Reference" "#PWR0405" (id 0) (at 139.7 162.56 0)
       (effects (font (size 1.27 1.27)) hide)
     )
@@
   (symbol (lib_id "Device:C_Small") (at 120.65 165.1 0) (unit 1)
     (in_bom yes) (on_board yes) (fields_autoplaced)
-    (property "Reference" "C4002" (id 0) (at 123.19 163.8362 0)
+    (property "Reference" "C402" (id 0) (at 123.19 163.8362 0)
       (effects (font (size 1.27 1.27)) (justify left))
     )
@@
   (symbol (lib_id "power:+3.3V") (at 207.01 58.42 90) (unit 1)
     (in_bom yes) (on_board yes) (fields_autoplaced)
-    (property "Reference" "#PWR0131" (id 0) (at 210.82 58.42 0)
+    (property "Reference" "#PWR0407" (id 0) (at 210.82 58.42 0)
       (effects (font (size 1.27 1.27)) hide)
     )
@@
   (symbol (lib_id "power:+3.3V") (at 242.57 58.42 270) (mirror x) (unit 1)
     (in_bom yes) (on_board yes) (fields_autoplaced)
-    (property "Reference" "#PWR0133" (id 0) (at 238.76 58.42 0)
+    (property "Reference" "#PWR0409" (id 0) (at 238.76 58.42 0)
       (effects (font (size 1.27 1.27)) hide)
     )
@@
   (symbol (lib_id "power:+3.3V") (at 35.56 166.37 90) (unit 1)
     (in_bom yes) (on_board yes) (fields_autoplaced)
-    (property "Reference" "#PWR0124" (id 0) (at 39.37 166.37 0)
+    (property "Reference" "#PWR0402" (id 0) (at 39.37 166.37 0)
       (effects (font (size 1.27 1.27)) hide)
     )
@@
   (symbol (lib_id "Connector:Conn_01x07_Female") (at 237.49 63.5 0) (mirror y) (unit 1)
     (in_bom yes) (on_board yes)
-    (property "Reference" "J4006" (id 0) (at 231.14 62.23 0))
+    (property "Reference" "J406" (id 0) (at 231.14 62.23 0))
     (property "Value" "tofDroit" (id 1) (at 231.14 64.77 0))
     (property "Footprint" "Connector_JST:JST_XH_B7B-XH-A_1x07_P2.50mm_Vertical" (id 2) (at 237.49 63.5 0)
@@
   (symbol (lib_id "power:GND") (at 35.56 161.29 270) (unit 1)
     (in_bom yes) (on_board yes) (fields_autoplaced)
-    (property "Reference" "#PWR0125" (id 0) (at 29.21 161.29 0)
-      (effects (font (size 1.27 1.27)) hide)
-    )
+    (property "Reference" "#PWR0401" (id 0) (at 29.21 161.29 0)
+      (effects (font (size 1.27 1.27)) hide)
+    )

Commit message: Routing
Parts:
- added R401, R402, R403, R404: 2.2k, Resistor_SMD:R_0603_1608Metric_Pad0.98x0.95mm_HandSolder, symbol Device:R_Small
Connections:
- net +3.3V: now also R401.1, R402.1, R403.1, R404.1; no longer J402.1 (Pin_1)
- net TOF1_SCL: now also R403.2
- net TOF1_SDA: now also R404.2
- net TOF2_SCL: now also R401.2
- net TOF2_SDA: now also R402.2
- new net +5V: J402.1 (Pin_1)
Other:
- note added: "pull up"
