File: Projet/stm32f070rb_sch.kicad_sch (KiCad schematic)
At the start: 21 parts, among them J201 Conn_02x07_Odd_Even, U201 STM32G070RBT6, Y201 16 MHz

Commit message: PCB_FINAL
Parts:
- removed C205: 100nF, Capacitor_SMD:C_0603_1608Metric_Pad1.08x0.95mm_HandSolder, symbol Device:C_Small
Connections:
- net OPTQ1: now also U201.1 (PC11); no longer U201.14 (PC1)
- net OSC_IN: now reaches C203.1, U201.10 (PF0-OSC_IN), Y201.3
- net OSC_OUT: now reaches R203.1, U201.11 (PF1-OSC_OUT)
- net ESP_EN: no longer names the net of U201.21 (PA4)
- no-connect marks 28 -> 29
Changed lines of the file:
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@@
   (junction (at 234.95 59.69) (diameter 0) (color 0 0 0 0)
-  )
-  (junction (at 246.38 46.99) (diameter 0) (color 0 0 0 0)
-  )
-  (junction (at 246.38 59.69) (diameter 0) (color 0 0 0 0)
   )
   (junction (at 137.16 100.33) (diameter 0) (color 0 0 0 0)
@@
   (no_connect (at 58.42 86.36))
   (no_connect (at 243.84 120.65))
+  (no_connect (at 58.42 48.26))
   (no_connect (at 243.84 128.27))
   (no_connect (at 58.42 50.8))
@@
   (no_connect (at 109.22 55.88))
   (no_connect (at 109.22 63.5))
-  (no_connect (at 109.22 60.96))
+  (no_connect (at 109.22 35.56))
   (no_connect (at 109.22 38.1))
   (no_connect (at 58.42 93.98))
@@
     (stroke (width 0) (type default) (color 0 0 0 0))
   )
-  (wire (pts (xy 246.38 59.69) (xy 246.38 55.88))
-    (stroke (width 0) (type default) (color 0 0 0 0))
-  )
   (wire (pts (xy 213.36 128.27) (xy 213.36 133.35))
     (stroke (width 0) (type default) (color 0 0 0 0))
@@
     (stroke (width 0) (type default) (color 0 0 0 0))
   )
-  (wire (pts (xy 257.81 46.99) (xy 246.38 46.99))
-    (stroke (width 0) (type default) (color 0 0 0 0))
-  )
   (wire (pts (xy 137.16 115.57) (xy 121.92 115.57))
     (stroke (width 0) (type default) (color 0 0 0 0))
@@
     (stroke (width 0) (type default) (color 0 0 0 0))
   )
-  (wire (pts (xy 246.38 46.99) (xy 234.95 46.99))
+  (wire (pts (xy 234.95 46.99) (xy 257.81 46.99))
     (stroke (width 0) (type default) (color 0 0 0 0))
   )
@@
     (stroke (width 0) (type default) (color 0 0 0 0))
   )
-  (wire (pts (xy 234.95 59.69) (xy 246.38 59.69))
+  (wire (pts (xy 234.95 59.69) (xy 257.81 59.69))
     (stroke (width 0) (type default) (color 0 0 0 0))
   )
@@
     (stroke (width 0) (type default) (color 0 0 0 0))
   )
-  (wire (pts (xy 246.38 50.8) (xy 246.38 46.99))
-    (stroke (width 0) (type default) (color 0 0 0 0))
-  )
   (wire (pts (xy 133.35 100.33) (xy 137.16 100.33))
     (stroke (width 0) (type default) (color 0 0 0 0))
@@
     (stroke (width 0) (type default) (color 0 0 0 0))
   )
-  (wire (pts (xy 257.81 59.69) (xy 246.38 59.69))
-    (stroke (width 0) (type default) (color 0 0 0 0))
-  )
   (wire (pts (xy 116.84 104.14) (xy 116.84 115.57))
     (stroke (width 0) (type default) (color 0 0 0 0))
@@
   )
   (wire (pts (xy 150.368 115.57) (xy 137.16 115.57))
-    (stroke (width 0) (type default) (color 0 0 0 0))
-  )
-  (wire (pts (xy 109.22 35.56) (xy 113.03 35.56))
     (stroke (width 0) (type default) (color 0 0 0 0))
   )
@@
     (effects (font (size 1.27 1.27)) (justify left bottom))
   )
+  (label "OSC_IN" (at 121.666 101.6 0)
+    (effects (font (size 1.27 1.27)) (justify left bottom))
+  )
   (label "ST_LINK_RX" (at 257.556 135.89 0)
     (effects (font (size 1.27 1.27)) (justify left bottom))
@@
   )
   (label "DRV_2_FWD_JP" (at 110.744 76.2 0)
+    (effects (font (size 1.27 1.27)) (justify left bottom))
+  )
+  (label "OSC_OUT" (at 115.062 104.14 0)
     (effects (font (size 1.27 1.27)) (justify left bottom))
   )
@@
     (effects (font (size 1.27 1.27)) (justify left))
   )
-  (hierarchical_label "OPTQ1" (shape input) (at 113.03 35.56 0)
+  (hierarchical_label "OPTQ1" (shape input) (at 109.22 60.96 0)
     (effects (font (size 1.27 1.27)) (justify left))
   )
@@
   (hierarchical_label "CLR_S0" (shape input) (at 109.22 81.28 0)
     (effects (font (size 1.27 1.27)) (justify left))
-  )
-  (hierarchical_label "ESP_EN" (shape input) (at 58.42 48.26 180)
-    (effects (font (size 1.27 1.27)) (justify right))
   )
   (hierarchical_label "CLR_OE" (shape input) (at 109.22 91.44 0)
@@
     (pin "1")
   )
-  (symbol (lib_id "Device:C_Small") (at 246.38 53.34 180) (unit 1)
-    (in_bom yes) (on_board yes) (fields_autoplaced)
-    (property "Reference" "C205" (id 0) (at 248.92 52.0635 0)
-      (effects (font (size 1.27 1.27)) (justify right))
-    )
-    (property "Value" "100nF" (id 1) (at 248.92 54.6035 0)
-      (effects (font (size 1.27 1.27)) (justify right))
-    )
-    (property "Footprint" "Capacitor_SMD:C_0603_1608Metric_Pad1.08x0.95mm_HandSolder" (id 2) (at 246.38 53.34 0)
-      (effects (font (size 1.27 1.27)) hide)
-    )
-    (property "Datasheet" "~" (id 3) (at 246.38 53.34 0)
-      (effects (font (size 1.27 1.27)) hide)
-    )
-    (pin "1")
-    (pin "2")
-  )
   (symbol (lib_id "Device:LED_Small") (at 90.17 168.91 90) (unit 1)
